File: Ma2 Keybaord/Ma2 Keybaord.kicad_pcb (KiCad board)
At the start: 2 copper layers, 97 parts, among them J1 Conn_01x05, J2 Conn_01x02, J4 Conn_01x02, J5 Conn_01x03, SW1 MX_SW_HS, SW10 MX_SW_HS, SW11 MX_SW_HS, SW12 MX_SW_HS, SW13 MX_SW_HS, SW14 MX_SW_HS, SW15 MX_SW_HS, SW16 MX_SW_HS, SW17 MX_SW_HS, SW18 MX_SW_HS, SW19 MX_SW_HS, SW2 MX_SW_HS, SW20 MX_SW_HS, SW21 MX_SW_HS, SW22 MX_SW_HS, SW23 MX_SW_HS, SW24 MX_SW_HS, SW25 MX_SW_HS, SW26 MX_SW_HS, SW27 MX_SW_HS, SW28 MX_SW_HS, SW29 MX_SW_HS, SW3 MX_SW_HS, SW30 MX_SW_HS, SW31 MX_SW_HS, SW32 MX_SW_HS, SW33 MX_SW_HS, SW34 MX_SW_HS, SW35 MX_SW_HS, SW36 MX_SW_HS, SW37 MX_SW_HS, SW38 MX_SW_HS, SW39 MX_SW_HS, SW4 MX_SW_HS, SW40 MX_SW_HS, SW41 MX_SW_HS, SW42 MX_SW_HS, SW43 MX_SW_HS, SW44 MX_SW_HS, SW45 MX_SW_HS, SW46 MX_SW_HS, SW47 MX_SW_HS, SW48 MX_SW_HS, SW49 MX_SW_HS, SW5 MX_SW_HS, SW50 MX_SW_HS, SW51 MX_SW_HS, SW52 MX_SW_HS, SW53 MX_SW_HS, SW54 MX_SW_HS, SW55 MX_SW_HS, SW56 MX_SW_HS, SW57 MX_SW_HS, SW58 MX_SW_HS, SW59 MX_SW_HS, SW6 MX_SW_HS, SW60 MX_SW_HS, SW61 MX_SW_HS, SW62 MX_SW_HS, SW63 MX_SW_HS, SW64 MX_SW_HS, SW65 MX_SW_HS, SW66 MX_SW_HS, SW67 MX_SW_HS, SW68 MX_SW_HS, SW69 MX_SW_HS, SW7 MX_SW_HS, SW70 MX_SW_HS, SW71 MX_SW_HS, SW72 MX_SW_HS, SW73 MX_SW_HS, SW74 MX_SW_HS, SW75 MX_SW_HS, SW76 MX_SW_HS, SW77 MX_SW_HS, SW8 MX_SW_HS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

Commit message: more work on the keyboard lay out on the PCB also making 4.5U stab
Parts:
- added SW64: MX_SW_HS, marbastlib-mx:SW_MX_HS_1u, F.Cu at (298.4, 132.6)
- S2: footprint marbastlib-mx:STAB_MX_P_2u -> marbastlib-mx:STAB_MX_P_2.25u
- S3: footprint marbastlib-mx:STAB_MX_P_6u -> marbastlib-mx:STAB_MX_4.5u
- SW31: footprint marbastlib-mx:SW_MX_HS_1u -> marbastlib-mx:SW_MX_HS_1.5u
- SW35, SW63: footprint marbastlib-mx:SW_MX_HS_1u -> marbastlib-mx:SW_MX_HS_1.75u
- SW51: footprint marbastlib-mx:SW_MX_HS_1u -> marbastlib-mx:SW_MX_HS_1.25u
- SW68: renamed from SW67; footprint marbastlib-mx:SW_MX_HS_1u -> marbastlib-mx:SW_MX_HS_1.5u
- SW69: renamed from SW68; footprint marbastlib-mx:SW_MX_HS_1u -> marbastlib-mx:SW_MX_HS_1.5u
- SW70: renamed from SW69; footprint marbastlib-mx:SW_MX_HS_1u -> marbastlib-mx:SW_MX_HS_1.5u
- SW71: renamed from SW70; footprint marbastlib-mx:SW_MX_HS_1u -> marbastlib-mx:SW_MX_HS_1.5u
- SW73: renamed from SW72; footprint marbastlib-mx:SW_MX_HS_1u -> marbastlib-mx:SW_MX_HS_1.5u
- SW75: renamed from SW74; footprint marbastlib-mx:SW_MX_HS_1u -> marbastlib-mx:SW_MX_HS_1.5u
- moved SW51 445.7 mm to (67.5, 132.6)
- moved SW21 439.8 mm to (131.8, 94.5)
- moved SW52 437.1 mm to (88.9, 132.6)
- moved SW39 400.5 mm to (155.6, 113.5)
- moved SW37 389.1 mm to (117.5, 113.5)
- moved SW56 376.8 mm to (165.1, 132.6)
- moved SW36 374.7 mm to (98.4, 113.5)
- moved SW69 366.8 mm to (69.8, 151.6)
- moved SW20 360.3 mm to (112.7, 94.5)
- moved SW19 359.6 mm to (93.7, 94.5)
- moved SW35 357.9 mm to (72.2, 113.5)
- moved SW24 350.0 mm to (188.9, 94.5)
- moved SW40 349.9 mm to (174.6, 113.5)
- moved SW72 335.8 mm to (189.7, 151.6)
- moved SW26 325.4 mm to (227.0, 94.5)
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- renumbered SW64 to SW65, SW65 to SW66, SW66 to SW67, SW71 to SW72, SW73 to SW74, SW75 to SW76, SW76 to SW77, SW77 to SW78
